Commit message: la simu commence a bien marché

File: braccio_arm_description/urdf/braccio_arm.urdf (robot description, URDF)
Before this commit: robot braccio_arm, 8 links, 7 joints
Joints:
- joint sub_gripper_joint: mimic joint=gripper_joint -> (none)

File: braccio_arm_description/urdf/braccio_arm.xacro (robot description, xacro)
@@ -30,6 +30,6 @@
         <inertial>
             <origin xyz="0 0 0" rpy="0 0 0"/>
-            <mass value="0.1"/>
-            <box_inertia m="0.1" x="0.1" y="0.1" z="0.1"/>
+            <mass value="0.05"/>
+            <box_inertia m="0.05" x="0.02" y="0.02" z="0.05"/>
         </inertial>
     </link>
@@ -44,6 +44,6 @@
         <inertial>
             <origin xyz="0 0 0" rpy="0 0 0"/>
-            <mass value="0.1"/>
-            <box_inertia m="0.1" x="0.1" y="0.1" z="0.1"/>
+            <mass value="0.05"/>
+            <box_inertia m="0.05" x="0.02" y="0.02" z="0.05"/>
         </inertial>
     </link>
@@ -58,6 +58,6 @@
         <inertial>
             <origin xyz="0 0 0" rpy="0 0 0"/>
-            <mass value="0.1"/>
-            <box_inertia m="0.1" x="0.1" y="0.1" z="0.1"/>
+            <mass value="0.05"/>
+            <box_inertia m="0.05" x="0.02" y="0.02" z="0.05"/>
         </inertial>
     </link>
@@ -72,6 +72,6 @@
         <inertial>
             <origin xyz="0 0 0" rpy="0 0 0"/>
-            <mass value="0.1"/>
-            <box_inertia m="0.1" x="0.1" y="0.1" z="0.1"/>
+            <mass value="0.05"/>
+            <box_inertia m="0.05" x="0.02" y="0.02" z="0.05"/>
         </inertial>
     </link>
@@ -86,6 +86,6 @@
         <inertial>
             <origin xyz="0 0 0" rpy="0 0 0"/>
-            <mass value="0.1"/>
-            <box_inertia m="0.1" x="0.1" y="0.1" z="0.1"/>
+            <mass value="0.05"/>
+            <box_inertia m="0.05" x="0.02" y="0.02" z="0.05"/>
         </inertial>
     </link>
@@ -100,6 +100,6 @@
         <inertial>
             <origin xyz="0 0 0" rpy="0 0 0"/>
-            <mass value="0.1"/>
-            <box_inertia m="0.1" x="0.1" y="0.1" z="0.1"/>
+            <mass value="0.05"/>
+            <box_inertia m="0.05" x="0.02" y="0.02" z="0.05"/>
         </inertial>
     </link>
@@ -110,13 +110,27 @@
             </geometry>
             <material name="white" />
-            <origin rpy="0 1.5708 0" xyz="0 -0.012 0" />
-        </visual>
-        <inertial>
-            <origin xyz="0 0 0" rpy="0 0 0"/>
-            <mass value="0.1"/>
-            <box_inertia m="0.1" x="0.1" y="0.1" z="0.1"/>
+            <origin rpy="0 1.5708 0" xyz="0 -0.007 0" />
+        </visual>
+        <visual>
+            <geometry>
+                <mesh filename="package://braccio_arm_description/stl/braccio_left_gripper.stl" scale="0.001 0.001 0.001" />
+            </geometry>
+            <material name="white" />
+            <origin rpy="0 1.5708 0" xyz="0 -0.017 0" />
+        </visual>
+        <inertial>
+            <origin xyz="0 0 0" rpy="0 0 0"/>
+            <mass value="0.01"/>
+            <box_inertia m="0.01" x="0.02" y="0.02" z="0.05"/>
         </inertial>
     </link>
     <link name="right_gripper_link">
+        <collision>
+            <geometry>
+                <cylinder length="0.01" radius=".053" />
+            </geometry>
+            <material name="black" />
+            <origin rpy="0 0 0" xyz="0 0 0" />
+        </collision>
         <visual>
             <geometry>
@@ -124,10 +138,17 @@
             </geometry>
             <material name="white" />
-            <origin rpy="0 1.5708 0" xyz="0 -0.012 0.010" />
-        </visual>
-        <inertial>
-            <origin xyz="0 0 0" rpy="0 0 0"/>
-            <mass value="0.1"/>
-            <box_inertia m="0.1" x="0.1" y="0.1" z="0.1"/>
+            <origin rpy="0 1.5708 0" xyz="0 -0.017 0.010" />
+        </visual>
+        <visual>
+            <geometry>
+                <mesh filename="package://braccio_arm_description/stl/braccio_right_gripper.stl" scale="0.001 0.001 0.001" />
+            </geometry>
+            <material name="white" />
+            <origin rpy="0 1.5708 0" xyz="0 -0.007 0.010" />
+        </visual>
+        <inertial>
+            <origin xyz="0 0 0" rpy="0 0 0"/>
+            <mass value="0.01"/>
+            <box_inertia m="0.01" x="0.02" y="0.02" z="0.05"/>
         </inertial>
     </link>
@@ -177,5 +198,5 @@
         <axis xyz="0 1 0" />
         <mimic joint="gripper_joint" />
-        <limit effort="1000.0" lower="1.2741" upper="2.3732" velocity="1.0" />
+        <limit effort="1000.0" lower="0.1750" upper="1.2741" velocity="1.0" />
         <origin rpy="0 3.4383 0" xyz="-0.010 0 0.03" />
         <parent link="wrist_roll_link" />
