Commit message: simu avec collision ok

File: braccio_arm_description/urdf/braccio_arm.xacro (robot description, xacro)
@@ -35,4 +35,11 @@
     </link>
     <link name="braccio_arm_base_link">
+        <collision>
+            <geometry>
+                <cylinder length="0.06" radius="0.04"/>
+            </geometry>
+            <material name="black" />
+            <origin rpy="0 0 0" xyz="0 0 0.03" />
+        </collision>
         <visual>
             <geometry>
@@ -49,4 +56,11 @@
     </link>
     <link name="shoulder_link">
+        <collision>
+            <geometry>
+                <cylinder length="0.10" radius="0.03"/>
+            </geometry>
+            <material name="black" />
+            <origin rpy="0 0 0" xyz="0 0 0.05" />
+        </collision>
         <visual>
             <geometry>
@@ -63,4 +77,11 @@
     </link>
     <link name="elbow_link">
+        <collision>
+            <geometry>
+                <cylinder length="0.10" radius="0.03"/>
+            </geometry>
+            <material name="black" />
+            <origin rpy="0 0 0" xyz="0 0 0.05" />
+        </collision>
         <visual>
             <geometry>
@@ -91,4 +112,11 @@
     </link>
     <link name="wrist_roll_link">
+        <collision>
+            <geometry>
+                <cylinder length="0.08" radius="0.025"/>
+            </geometry>
+            <material name="black" />
+            <origin rpy="0 0 0" xyz="0 0 -0.02" />
+        </collision>
         <visual>
             <geometry>
@@ -105,4 +133,11 @@
     </link>
     <link name="left_gripper_link">
+        <collision>
+            <geometry>
+                <box size="0.1 0.02 0.01"/>
+            </geometry>
+            <material name="black" />
+            <origin rpy="0 0 0" xyz="0.04 0 0" />
+        </collision>
         <visual>
             <geometry>
@@ -128,8 +163,8 @@
         <collision>
             <geometry>
-                <cylinder length="0.01" radius=".053" />
-            </geometry>
-            <material name="black" />
-            <origin rpy="0 0 0" xyz="0 0 0" />
+                <box size="0.1 0.02 0.01"/>
+            </geometry>
+            <material name="black" />
+            <origin rpy="0 0 0" xyz="0.04 0 0" />
         </collision>
         <visual>

Commit message: ajout de cube

File: braccio_arm_description/urdf/braccio_arm.xacro (robot description, xacro)
@@ -1,9 +1,9 @@
 <?xml version="1.0"?>
 <robot name="braccio_arm" xmlns:xacro="http://www.ros.org/wiki/xacro">
-      <macro name="box_inertia" params="m x y z">
+      <xacro:macro name="box_inertia" params="m x y z">
         <inertia  ixx="${m*(y*y+z*z)/12}" ixy = "0" ixz = "0"
                   iyy="${m*(x*x+z*z)/12}" iyz = "0"
                   izz="${m*(x*x+z*z)/12}" />
-      </macro>
+      </xacro:macro>
     <material name="orange">
         <color rgba="0.57 0.17 0.0 1" />

Commit message: simulation et grasping des cubes réalistes

File: braccio_arm_description/urdf/braccio_arm.xacro (robot description, xacro)
@@ -135,15 +135,22 @@
         <collision>
             <geometry>
-                <box size="0.1 0.02 0.01"/>
-            </geometry>
-            <material name="black" />
-            <origin rpy="0 0 0" xyz="0.04 0 0" />
-        </collision>
-        <visual>
+                <box size="0.05 0.02 0.01"/>
+            </geometry>
+            <material name="black" />
+            <origin rpy="0 -1.5708 0" xyz="0 0 -0.025" />
+        </collision>
+        <visual>
+            <geometry>
+                <box size="0.05 0.02 0.01"/>
+            </geometry>
+            <material name="black" />
+            <origin rpy="0 -1.5708 0" xyz="0 0 -0.025" />
+        </visual>
+<!--        <visual>
             <geometry>
                 <mesh filename="package://braccio_arm_description/stl/braccio_left_gripper.stl" scale="0.001 0.001 0.001" />
             </geometry>
             <material name="white" />
-            <origin rpy="0 1.5708 0" xyz="0 -0.007 0" />
+            <origin rpy="0 0 0" xyz="0 -0.007 0" />
         </visual>
         <visual>
@@ -152,10 +159,10 @@
             </geometry>
             <material name="white" />
-            <origin rpy="0 1.5708 0" xyz="0 -0.017 0" />
-        </visual>
+            <origin rpy="0 0 0" xyz="0 -0.017 0" />
+        </visual>        -->
         <inertial>
             <origin xyz="0 0 0" rpy="0 0 0"/>
             <mass value="0.01"/>
-            <box_inertia m="0.01" x="0.02" y="0.02" z="0.05"/>
+            <box_inertia m="0.01" x="0.01" y="0.025" z="0.005"/>
         </inertial>
     </link>
@@ -163,15 +170,22 @@
         <collision>
             <geometry>
-                <box size="0.1 0.02 0.01"/>
-            </geometry>
-            <material name="black" />
-            <origin rpy="0 0 0" xyz="0.04 0 0" />
-        </collision>
-        <visual>
+                <box size="0.05 0.02 0.01"/>
+            </geometry>
+            <material name="black" />
+            <origin rpy="0 -1.5708 0" xyz="0 0 -0.025" />
+        </collision>
+        <visual>
+            <geometry>
+                <box size="0.05 0.02 0.01"/>
+            </geometry>
+            <material name="black" />
+            <origin rpy="0 -1.5708 0" xyz="0 0 -0.025" />
+        </visual>
+<!--        <visual>
             <geometry>
                 <mesh filename="package://braccio_arm_description/stl/braccio_right_gripper.stl" scale="0.001 0.001 0.001" />
             </geometry>
             <material name="white" />
-            <origin rpy="0 1.5708 0" xyz="0 -0.017 0.010" />
+            <origin rpy="0 0 0" xyz="0 -0.017 0.010" />
         </visual>
         <visual>
@@ -180,10 +194,10 @@
             </geometry>
             <material name="white" />
-            <origin rpy="0 1.5708 0" xyz="0 -0.007 0.010" />
-        </visual>
+            <origin rpy="0 0 0" xyz="0 -0.007 0.010" />
+        </visual>   -->
         <inertial>
             <origin xyz="0 0 0" rpy="0 0 0"/>
             <mass value="0.01"/>
-            <box_inertia m="0.01" x="0.02" y="0.02" z="0.05"/>
+            <box_inertia m="0.01" x="0.01" y="0.025" z="0.005"/>
         </inertial>
     </link>
@@ -218,21 +232,21 @@
     <joint name="wrist_roll_joint" type="revolute">
         <axis xyz="0 0 -1" />
-        <limit effort="1000.0" lower="0.0" upper="3.1416" velocity="1.0" />
+        <limit effort="1000.0" lower="0" upper="3.1416" velocity="1.0" />
         <origin rpy="0 0 1.5708" xyz="0 0.0 0.06" />
         <parent link="wrist_pitch_link" />
         <child link="wrist_roll_link" />
     </joint>
-    <joint name="gripper_joint" type="revolute">
-        <axis xyz="0 -1 0" />
-        <limit effort="1000.0" lower="0.1750" upper="1.2741" velocity="1.0" />
-        <origin rpy="0 -0.2967 0" xyz="0.010 0 0.03" />
+    <joint name="gripper_joint" type="prismatic">
+        <axis xyz="-1 0 0" />
+        <limit effort="1000.0" lower="0.02" upper="0.07" velocity="1.0" />
+        <origin rpy="0 0 0" xyz="0.010 0 0.08" />
         <parent link="wrist_roll_link" />
         <child link="right_gripper_link" />
     </joint>
-    <joint name="sub_gripper_joint" type="revolute">
-        <axis xyz="0 1 0" />
+    <joint name="sub_gripper_joint" type="prismatic">
+        <axis xyz="1 0 0" />
         <mimic joint="gripper_joint" />
-        <limit effort="1000.0" lower="0.1750" upper="1.2741" velocity="1.0" />
-        <origin rpy="0 3.4383 0" xyz="-0.010 0 0.03" />
+        <limit effort="1000.0" lower="0.02" upper="0.07" velocity="1.0" />
+        <origin rpy="0 0 0" xyz="-0.010 0 0.08" />
         <parent link="wrist_roll_link" />
         <child link="left_gripper_link" />

File: braccio_arm_gazebo/urdf/cube.xacro (robot description, xacro)
@@ -5,5 +5,5 @@
       <origin xyz="0 0 0" />
       <mass value="${m}" />
-      <inertia  ixx="1.0" ixy="0.0"  ixz="0.0"  iyy="100.0"  iyz="0.0"  izz="1.0" />
+      <inertia  ixx="${m*m/12.0}" ixy="0.0"  ixz="0.0"  iyy="${m*m/12.0}"  iyz="0.0"  izz="${m*m/12.0}" />
     </inertial>
     <visual>

Commit message: update the marker

File: braccio_arm_description/urdf/braccio_arm.xacro (robot description, xacro)
@@ -17,6 +17,7 @@
   <link name="world"/>
   <joint name="fixed" type="fixed">
-    <parent link="world"/>
-    <child link="base_link"/>
+        <origin xyz="0 0 0.01" rpy="0 0 0"/>
+        <parent link="world"/>
+        <child link="base_link"/>
   </joint>
     <link name="base_link">
@@ -201,4 +202,28 @@
             <box_inertia m="0.01" x="0.01" y="0.025" z="0.005"/>
         </inertial>
+    </link>
+    <link name="camera_link">
+        <inertial>
+            <mass value="0.01" />
+            <origin xyz="0 0 0" />
+            <inertia ixx="0.001"  ixy="0.0"  ixz="0.0"
+                    iyy="0.001"  iyz="0.0"
+                    izz="0.001" />
+        </inertial>
+        <visual>
+            <origin xyz="0 0 0" rpy="0 0 0"/>
+            <geometry>
+                <box size="0.02 0.10 0.02" />
+            </geometry>
+            <material name="Cyan">
+                <color rgba="0 1.0 1.0 1.0"/>
+            </material>
+        </visual>
+        <collision>
+            <origin xyz="0 0 0" rpy="0 0 0"/>
+            <geometry>
+                <box size="0.02 0.1 0.02" />
+            </geometry>
+        </collision>
     </link>
     <joint name="base_joint" type="revolute">
@@ -252,4 +277,9 @@
         <child link="left_gripper_link" />
     </joint>
+    <joint name="camera_joint" type="fixed">
+        <origin xyz="0 0.04 0" rpy="-1.57 -1.57 0" />
+        <parent link="wrist_roll_link" />
+        <child link="camera_link"/>
+    </joint>
     <xacro:include filename="$(find braccio_arm_description)/urdf/braccio_arm.gazebo" />
 </robot>

File: braccio_arm_gazebo/urdf/cube1.xacro (robot description, xacro)
@@ -3,5 +3,5 @@
     <xacro:include filename="$(find braccio_arm_gazebo)/urdf/cube.xacro" />
     <link name="my_box">
-        <aruco_cube t1="10" t2="11" t3="12" t4="13" t5="14" t6="15" dim="0.05" m="0.05"/>
+        <aruco_cube t1="10" t2="11" t3="12" t4="13" t5="14" t6="15" dim="1" m="0.05"/>
     </link>
     <gazebo reference="my_box">

Commit message: update the challenges

File: braccio_arm_description/urdf/braccio_arm.xacro (robot description, xacro)
@@ -1,9 +1,9 @@
 <?xml version="1.0"?>
 <robot name="braccio_arm" xmlns:xacro="http://www.ros.org/wiki/xacro">
-      <xacro:macro name="box_inertia" params="m x y z">
+      <macro name="box_inertia" params="m x y z">
         <inertia  ixx="${m*(y*y+z*z)/12}" ixy = "0" ixz = "0"
                   iyy="${m*(x*x+z*z)/12}" iyz = "0"
                   izz="${m*(x*x+z*z)/12}" />
-      </xacro:macro>
+      </macro>
     <material name="orange">
         <color rgba="0.57 0.17 0.0 1" />
@@ -282,4 +282,4 @@
         <child link="camera_link"/>
     </joint>
-    <xacro:include filename="$(find braccio_arm_description)/urdf/braccio_arm.gazebo" />
+    <include filename="$(find braccio_arm_description)/urdf/braccio_arm.gazebo" />
 </robot>

File: braccio_challenge/urdf/basket.xacro (robot description, xacro)
@@ -1,5 +1,5 @@
 <?xml version="1.0"?>
 <robot xmlns:xacro="http://www.ros.org/wiki/xacro">
- <xacro:macro name="aruco_basket" params="t1 t2 t3 t4 t5 l w h dim_marker m ">
+ <macro name="aruco_basket" params="t1 t2 t3 t4 l w h dim_marker m ">
    <inertial>
       <origin xyz="0 0 0" />
@@ -79,4 +79,4 @@
       </geometry>
     </collision>
-</xacro:macro>
+</macro>
 </robot>

File: braccio_challenge/urdf/basket1.xacro (robot description, xacro)
@@ -1,5 +1,5 @@
 <?xml version="4.0"?>
 <robot xmlns:xacro="http://www.ros.org/wiki/xacro">
-    <xacro:include filename="$(find braccio_challenge)/urdf/basket.xacro" />
+    <include filename="$(find braccio_challenge)/urdf/basket.xacro" />
     <link name="world"/>
     <joint name="fixed" type="fixed">
@@ -9,5 +9,5 @@
     </joint>
     <link name="my_box">
-        <aruco_basket t1="0" t2="1" t3="2" t4="3" t5="4" l="0.15" w="0.15" h="0.15" dim_marker="0.05" m="0.05"/>
+        <aruco_basket t1="0" t2="1" t3="2" t4="3" l="0.15" w="0.15" h="0.15" dim_marker="0.05" m="0.05"/>
     </link>
     <gazebo reference="my_box">

File: braccio_challenge/urdf/basket2.xacro (robot description, xacro)
@@ -1,5 +1,5 @@
 <?xml version="4.0"?>
 <robot xmlns:xacro="http://www.ros.org/wiki/xacro">
-    <xacro:include filename="$(find braccio_challenge)/urdf/basket.xacro" />
+    <include filename="$(find braccio_challenge)/urdf/basket.xacro" />
     <link name="world"/>
     <joint name="fixed" type="fixed">
@@ -9,5 +9,5 @@
     </joint>
     <link name="my_box">
-        <aruco_basket t1="0" t2="1" t3="2" t4="3" t5="4" l="0.1" w="0.11" h="0.1" dim_marker="0.05" m="0.05"/>
+        <aruco_basket t1="5" t2="6" t3="7" t4="8"  l="0.1" w="0.1" h="0.1" dim_marker="0.05" m="0.05"/>
     </link>
     <gazebo reference="my_box">

Commit message: can run separately extern camera and robot

File: braccio_arm_description/urdf/braccio_arm.xacro (robot description, xacro)
@@ -1,9 +1,9 @@
 <?xml version="1.0"?>
 <robot name="braccio_arm" xmlns:xacro="http://www.ros.org/wiki/xacro">
-      <macro name="box_inertia" params="m x y z">
+      <xacro:macro name="box_inertia" params="m x y z">
         <inertia  ixx="${m*(y*y+z*z)/12}" ixy = "0" ixz = "0"
                   iyy="${m*(x*x+z*z)/12}" iyz = "0"
                   izz="${m*(x*x+z*z)/12}" />
-      </macro>
+      </xacro:macro>
     <material name="orange">
         <color rgba="0.57 0.17 0.0 1" />
@@ -203,5 +203,5 @@
         </inertial>
     </link>
-    <link name="camera_link">
+<!--    <link name="camera_link">
         <inertial>
             <mass value="0.01" />
@@ -226,5 +226,5 @@
             </geometry>
         </collision>
-    </link>
+    </link>-->
     <joint name="base_joint" type="revolute">
         <axis xyz="0 0 1" />
@@ -277,9 +277,9 @@
         <child link="left_gripper_link" />
     </joint>
-    <joint name="camera_joint" type="fixed">
+<!--    <joint name="camera_joint" type="fixed">
         <origin xyz="0 0.04 0" rpy="-1.57 -1.57 0" />
         <parent link="wrist_roll_link" />
         <child link="camera_link"/>
-    </joint>
-    <include filename="$(find braccio_arm_description)/urdf/braccio_arm.gazebo" />
+    </joint>    -->
+    <xacro:include filename="$(find braccio_arm_description)/urdf/braccio_arm.gazebo" />
 </robot>

File: braccio_challenge/urdf/basket.xacro (robot description, xacro)
@@ -1,5 +1,5 @@
 <?xml version="1.0"?>
 <robot xmlns:xacro="http://www.ros.org/wiki/xacro">
- <macro name="aruco_basket" params="t1 t2 t3 t4 l w h dim_marker m ">
+ <xacro:macro name="aruco_basket" params="t1 t2 t3 t4 l w h dim_marker m ">
    <inertial>
       <origin xyz="0 0 0" />
@@ -79,4 +79,4 @@
       </geometry>
     </collision>
-</macro>
+</xacro:macro>
 </robot>

File: braccio_challenge/urdf/basket1.xacro (robot description, xacro)
@@ -1,5 +1,5 @@
 <?xml version="4.0"?>
 <robot xmlns:xacro="http://www.ros.org/wiki/xacro">
-    <include filename="$(find braccio_challenge)/urdf/basket.xacro" />
+    <xacro:include filename="$(find braccio_challenge)/urdf/basket.xacro" />
     <link name="world"/>
     <joint name="fixed" type="fixed">

File: braccio_challenge/urdf/basket2.xacro (robot description, xacro)
@@ -1,5 +1,5 @@
 <?xml version="4.0"?>
 <robot xmlns:xacro="http://www.ros.org/wiki/xacro">
-    <include filename="$(find braccio_challenge)/urdf/basket.xacro" />
+    <xacro:include filename="$(find braccio_challenge)/urdf/basket.xacro" />
     <link name="world"/>
     <joint name="fixed" type="fixed">

Commit message: le probleme est qu'il faut changer robot_description quelque part

File: braccio_arm_description/urdf/braccio_arm.xacro (robot description, xacro)
@@ -203,5 +203,5 @@
         </inertial>
     </link>
-<!--    <link name="camera_link">
+ <!--   <link name="camera_link">
         <inertial>
             <mass value="0.01" />

File: braccio_camera_description/urdf/braccio_camera.xacro (robot description, xacro)
@@ -1,4 +1,4 @@
 <?xml version="1.0"?>
-<robot name="braccio_camera" xmlns:xacro="http://www.ros.org/wiki/xacro">
+<robot name="camera" xmlns:xacro="http://www.ros.org/wiki/xacro">
   <link name="world"/>
     <link name="body1">
@@ -53,5 +53,5 @@
         </collision>-->
     </link>
-    <joint name="base_joint" type="revolute">
+    <joint name="rotate" type="revolute">
         <axis xyz="0 0 1" />
         <limit effort="20.0" lower="-100.0" upper="100" velocity="0.1" />
@@ -60,5 +60,5 @@
         <child link="body1" />
     </joint>
-    <joint name="base_depth" type="prismatic">
+    <joint name="depth" type="prismatic">
         <axis xyz="1 0 0" />
         <limit effort="20.0" lower="00.0" upper="100" velocity="0.1" />
@@ -67,5 +67,5 @@
         <child link="body2" />
     </joint>
-    <joint name="base_height" type="prismatic">
+    <joint name="height" type="prismatic">
         <axis xyz="0 0 1" />
         <limit effort="20.0" lower="00.0" upper="100" velocity="0.1" />
@@ -74,5 +74,5 @@
         <child link="body3" />
     </joint>
-    <joint name="camera_tilt" type="revolute">
+    <joint name="tilt" type="revolute">
         <axis xyz="0 1 0" />
         <limit effort="2.0" lower="-3.14" upper="3.14" velocity="0.1" />
