Commit message: wip

File: braccio_arm_description/urdf/braccio_arm_and_camera.xacro (robot description, xacro)
@@ -34,4 +34,40 @@
             <box_inertia m="0.05" x="0.02" y="0.02" z="0.05"/>
         </inertial>
+    <visual>
+      <origin xyz="-0.1 0.055 -0.01" rpy="0 1.57 0"/>
+      <geometry>
+        <mesh filename="package://braccio_arm_gazebo/urdf/marker100/meshes/Marker100.dae" scale="1.0 0.1 0.1"/>
+      </geometry>
+    </visual>
+    <visual>
+      <origin xyz="-0.1 -0.055 -0.01" rpy="0 1.57 0"/>
+      <geometry>
+        <mesh filename="package://braccio_arm_gazebo/urdf/marker101/meshes/Marker101.dae" scale="1.0 0.1 0.1"/>
+      </geometry>
+    </visual>
+    <visual>
+      <origin xyz="-0.035 0.09 -0.01" rpy="0 1.57 0"/>
+      <geometry>
+        <mesh filename="package://braccio_arm_gazebo/urdf/marker102/meshes/Marker102.dae" scale="1.0 0.1 0.1"/>
+      </geometry>
+    </visual>
+    <visual>
+      <origin xyz="0.06 0.055 -0.01" rpy="0 1.57 0"/>
+      <geometry>
+        <mesh filename="package://braccio_arm_gazebo/urdf/marker103/meshes/Marker103.dae" scale="1.0 0.1 0.1"/>
+      </geometry>
+    </visual>
+    <visual>
+      <origin xyz="0.06 -0.055 -0.01" rpy="0 1.57 0"/>
+      <geometry>
+        <mesh filename="package://braccio_arm_gazebo/urdf/marker104/meshes/Marker104.dae" scale="1.0 0.1 0.1"/>
+      </geometry>
+    </visual>
+    <visual>
+      <origin xyz="-0.035 -0.09 -0.01" rpy="0 1.57 0"/>
+      <geometry>
+        <mesh filename="package://braccio_arm_gazebo/urdf/marker105/meshes/Marker105.dae" scale="1.0 0.1 0.1"/>
+      </geometry>
+    </visual>
     </link>
     <link name="braccio_arm_base_link">
@@ -203,5 +239,5 @@
         </inertial>
     </link>
- <!--   <link name="camera_link">
+    <link name="camera_embedded_link">
         <inertial>
             <mass value="0.01" />
@@ -226,5 +262,5 @@
             </geometry>
         </collision>
-    </link>-->
+    </link>
     <joint name="base_joint" type="revolute">
         <axis xyz="0 0 1" />
@@ -277,9 +313,9 @@
         <child link="left_gripper_link" />
     </joint>
-<!--    <joint name="camera_joint" type="fixed">
+    <joint name="camera_joint" type="fixed">
         <origin xyz="0 0.04 0" rpy="-1.57 -1.57 0" />
         <parent link="wrist_roll_link" />
-        <child link="camera_link"/>
-    </joint>    -->
+        <child link="camera_embedded_link"/>
+    </joint>
       <link name="camera_body1">
         <inertial>
@@ -333,5 +369,5 @@
         <axis xyz="0 0 1" />
         <limit effort="20.0" lower="-100.0" upper="100" velocity="0.1" />
-        <origin rpy="0 0 0" xyz="0 0 0" />
+        <origin rpy="0 0 3.14" xyz="0 0 0" />
         <parent link="world" />
         <child link="camera_body1" />

Commit message: ajout des messages

File: braccio_arm_description/urdf/braccio_arm_and_camera.xacro (robot description, xacro)
@@ -184,18 +184,4 @@
             <origin rpy="0 -1.5708 0" xyz="0 0 -0.025" />
         </visual>
-<!--        <visual>
-            <geometry>
-                <mesh filename="package://braccio_arm_description/stl/braccio_left_gripper.stl" scale="0.001 0.001 0.001" />
-            </geometry>
-            <material name="white" />
-            <origin rpy="0 0 0" xyz="0 -0.007 0" />
-        </visual>
-        <visual>
-            <geometry>
-                <mesh filename="package://braccio_arm_description/stl/braccio_left_gripper.stl" scale="0.001 0.001 0.001" />
-            </geometry>
-            <material name="white" />
-            <origin rpy="0 0 0" xyz="0 -0.017 0" />
-        </visual>        -->
         <inertial>
             <origin xyz="0 0 0" rpy="0 0 0"/>
@@ -219,18 +205,4 @@
             <origin rpy="0 -1.5708 0" xyz="0 0 -0.025" />
         </visual>
-<!--        <visual>
-            <geometry>
-                <mesh filename="package://braccio_arm_description/stl/braccio_right_gripper.stl" scale="0.001 0.001 0.001" />
-            </geometry>
-            <material name="white" />
-            <origin rpy="0 0 0" xyz="0 -0.017 0.010" />
-        </visual>
-        <visual>
-            <geometry>
-                <mesh filename="package://braccio_arm_description/stl/braccio_right_gripper.stl" scale="0.001 0.001 0.001" />
-            </geometry>
-            <material name="white" />
-            <origin rpy="0 0 0" xyz="0 -0.007 0.010" />
-        </visual>   -->
         <inertial>
             <origin xyz="0 0 0" rpy="0 0 0"/>

Commit message: change robot marqueur id

File: braccio_arm_description/urdf/braccio_arm_and_camera.xacro (robot description, xacro)
@@ -37,5 +37,5 @@
       <origin xyz="-0.1 0.055 -0.01" rpy="0 1.57 0"/>
       <geometry>
-        <mesh filename="package://braccio_arm_gazebo/urdf/marker100/meshes/Marker100.dae" scale="1.0 0.1 0.1"/>
+        <mesh filename="package://braccio_arm_gazebo/urdf/marker09/meshes/Marker09.dae" scale="1.0 0.1 0.1"/>
       </geometry>
     </visual>
@@ -43,5 +43,5 @@
       <origin xyz="-0.1 -0.055 -0.01" rpy="0 1.57 0"/>
       <geometry>
-        <mesh filename="package://braccio_arm_gazebo/urdf/marker101/meshes/Marker101.dae" scale="1.0 0.1 0.1"/>
+        <mesh filename="package://braccio_arm_gazebo/urdf/marker19/meshes/Marker19.dae" scale="1.0 0.1 0.1"/>
       </geometry>
     </visual>
@@ -49,5 +49,5 @@
       <origin xyz="-0.035 0.09 -0.01" rpy="0 1.57 0"/>
       <geometry>
-        <mesh filename="package://braccio_arm_gazebo/urdf/marker102/meshes/Marker102.dae" scale="1.0 0.1 0.1"/>
+        <mesh filename="package://braccio_arm_gazebo/urdf/marker29/meshes/Marker29.dae" scale="1.0 0.1 0.1"/>
       </geometry>
     </visual>
@@ -55,5 +55,5 @@
       <origin xyz="0.06 0.055 -0.01" rpy="0 1.57 0"/>
       <geometry>
-        <mesh filename="package://braccio_arm_gazebo/urdf/marker103/meshes/Marker103.dae" scale="1.0 0.1 0.1"/>
+        <mesh filename="package://braccio_arm_gazebo/urdf/marker39/meshes/Marker39.dae" scale="1.0 0.1 0.1"/>
       </geometry>
     </visual>
@@ -61,5 +61,5 @@
       <origin xyz="0.06 -0.055 -0.01" rpy="0 1.57 0"/>
       <geometry>
-        <mesh filename="package://braccio_arm_gazebo/urdf/marker104/meshes/Marker104.dae" scale="1.0 0.1 0.1"/>
+        <mesh filename="package://braccio_arm_gazebo/urdf/marker49/meshes/Marker49.dae" scale="1.0 0.1 0.1"/>
       </geometry>
     </visual>
@@ -67,5 +67,5 @@
       <origin xyz="-0.035 -0.09 -0.01" rpy="0 1.57 0"/>
       <geometry>
-        <mesh filename="package://braccio_arm_gazebo/urdf/marker105/meshes/Marker105.dae" scale="1.0 0.1 0.1"/>
+        <mesh filename="package://braccio_arm_gazebo/urdf/marker59/meshes/Marker59.dae" scale="1.0 0.1 0.1"/>
       </geometry>
     </visual>

Commit message: update the markers (back to previous version

File: braccio_arm_description/urdf/braccio_arm_and_camera.xacro (robot description, xacro)
@@ -37,5 +37,5 @@
       <origin xyz="-0.1 0.055 -0.01" rpy="0 1.57 0"/>
       <geometry>
-        <mesh filename="package://braccio_arm_gazebo/urdf/marker09/meshes/Marker09.dae" scale="1.0 0.1 0.1"/>
+        <mesh filename="package://braccio_arm_gazebo/urdf/marker100/meshes/Marker100.dae" scale="1.0 0.1 0.1"/>
       </geometry>
     </visual>
@@ -43,5 +43,5 @@
       <origin xyz="-0.1 -0.055 -0.01" rpy="0 1.57 0"/>
       <geometry>
-        <mesh filename="package://braccio_arm_gazebo/urdf/marker19/meshes/Marker19.dae" scale="1.0 0.1 0.1"/>
+        <mesh filename="package://braccio_arm_gazebo/urdf/marker101/meshes/Marker101.dae" scale="1.0 0.1 0.1"/>
       </geometry>
     </visual>
@@ -49,5 +49,5 @@
       <origin xyz="-0.035 0.09 -0.01" rpy="0 1.57 0"/>
       <geometry>
-        <mesh filename="package://braccio_arm_gazebo/urdf/marker29/meshes/Marker29.dae" scale="1.0 0.1 0.1"/>
+        <mesh filename="package://braccio_arm_gazebo/urdf/marker102/meshes/Marker102.dae" scale="1.0 0.1 0.1"/>
       </geometry>
     </visual>
@@ -55,5 +55,5 @@
       <origin xyz="0.06 0.055 -0.01" rpy="0 1.57 0"/>
       <geometry>
-        <mesh filename="package://braccio_arm_gazebo/urdf/marker39/meshes/Marker39.dae" scale="1.0 0.1 0.1"/>
+        <mesh filename="package://braccio_arm_gazebo/urdf/marker103/meshes/Marker103.dae" scale="1.0 0.1 0.1"/>
       </geometry>
     </visual>
@@ -61,5 +61,5 @@
       <origin xyz="0.06 -0.055 -0.01" rpy="0 1.57 0"/>
       <geometry>
-        <mesh filename="package://braccio_arm_gazebo/urdf/marker49/meshes/Marker49.dae" scale="1.0 0.1 0.1"/>
+        <mesh filename="package://braccio_arm_gazebo/urdf/marker104/meshes/Marker104.dae" scale="1.0 0.1 0.1"/>
       </geometry>
     </visual>
@@ -67,5 +67,5 @@
       <origin xyz="-0.035 -0.09 -0.01" rpy="0 1.57 0"/>
       <geometry>
-        <mesh filename="package://braccio_arm_gazebo/urdf/marker59/meshes/Marker59.dae" scale="1.0 0.1 0.1"/>
+        <mesh filename="package://braccio_arm_gazebo/urdf/marker105/meshes/Marker105.dae" scale="1.0 0.1 0.1"/>
       </geometry>
     </visual>
